Commit message: Add the controller to Gazebo and launch it in simulation

File: cp15_auxiliary_files/rb1_ros2_description/xacro/rb1_ros2_base.urdf.xacro (robot description, xacro)
@@ -84,5 +84,51 @@
 		<origin xyz="0.234 0.0 0.092" rpy="0 0 0"/>
 	</xacro:sensor_orbbec_astra>
-	<!-- Gazebo ros2 control plugins -->
-	<!-- <xacro:ros2_control/> -->
+    <!-- TRANSMISSION-->
+    <transmission name="left_wheel_transmission">
+        <type>transmission_interface/SimpleTransmission</type>
+        <joint name="$(arg prefix)left_wheel_joint">
+            <hardwareInterface>hardware_interface/VelocityJointInterface</hardwareInterface>
+        </joint>
+    </transmission>
+    <transmission name="right_wheel_transmission">
+        <type>transmission_interface/SimpleTransmission</type>
+        <joint name="$(arg prefix)right_wheel_joint">
+            <hardwareInterface>hardware_interface/VelocityJointInterface</hardwareInterface>
+        </joint>
+    </transmission>
+    <!-- <xacro:ros2_control/> -->
+    <ros2_control name="diff_drive" type="system">
+      <hardware>
+          <plugin>gazebo_ros2_control/GazeboSystem</plugin>
+      </hardware>
+      <joint name="$(arg prefix)left_wheel_joint">
+        <command_interface name="velocity">
+          <param name="min">-1</param>
+          <param name="max">1</param>
+        </command_interface>
+        <state_interface name="position"/>
+        <state_interface name="velocity"/>
+        <state_interface name="effort"/>
+      </joint>
+      <joint name="$(arg prefix)right_wheel_joint">
+        <command_interface name="velocity">
+          <param name="min">-1</param>
+          <param name="max">1</param>
+        </command_interface>
+        <state_interface name="position"/>
+        <state_interface name="velocity"/>
+        <state_interface name="effort"/>
+      </joint>
+    </ros2_control>
+    <!-- Gazebo ros2 control plugins -->
+    <gazebo>
+        <plugin filename="libgazebo_ros2_control.so" name="gazebo_ros2_control">
+            <parameters>$(find rb1_ros2_description)/config/rb1_controller.yaml</parameters>
+            <controller_manager_name>rb1_robot/controller_manager</controller_manager_name>
+            <ros>
+                <namespace>rb1_robot</namespace>
+                <remapping>/robot_description:=/rb1_robot/robot_description</remapping>
+            </ros>
+        </plugin>
+    </gazebo>
 </robot>

Commit message: Removed namespaces while working with one robot

File: cp15_auxiliary_files/rb1_ros2_description/xacro/rb1_ros2_base.urdf.xacro (robot description, xacro)
@@ -99,25 +99,25 @@
     <!-- <xacro:ros2_control/> -->
     <ros2_control name="diff_drive" type="system">
-      <hardware>
-          <plugin>gazebo_ros2_control/GazeboSystem</plugin>
-      </hardware>
-      <joint name="$(arg prefix)left_wheel_joint">
-        <command_interface name="velocity">
-          <param name="min">-1</param>
-          <param name="max">1</param>
-        </command_interface>
-        <state_interface name="position"/>
-        <state_interface name="velocity"/>
-        <state_interface name="effort"/>
-      </joint>
-      <joint name="$(arg prefix)right_wheel_joint">
-        <command_interface name="velocity">
-          <param name="min">-1</param>
-          <param name="max">1</param>
-        </command_interface>
-        <state_interface name="position"/>
-        <state_interface name="velocity"/>
-        <state_interface name="effort"/>
-      </joint>
+        <hardware>
+            <plugin>gazebo_ros2_control/GazeboSystem</plugin>
+        </hardware>
+        <joint name="$(arg prefix)left_wheel_joint">
+            <command_interface name="velocity">
+                <param name="min">-1</param>
+                <param name="max">1</param>
+            </command_interface>
+            <state_interface name="position"/>
+            <state_interface name="velocity"/>
+            <state_interface name="effort"/>
+        </joint>
+        <joint name="$(arg prefix)right_wheel_joint">
+            <command_interface name="velocity">
+                <param name="min">-1</param>
+                <param name="max">1</param>
+            </command_interface>
+            <state_interface name="position"/>
+            <state_interface name="velocity"/>
+            <state_interface name="effort"/>
+        </joint>
     </ros2_control>
     <!-- Gazebo ros2 control plugins -->
@@ -125,9 +125,4 @@
         <plugin filename="libgazebo_ros2_control.so" name="gazebo_ros2_control">
             <parameters>$(find rb1_ros2_description)/config/rb1_controller.yaml</parameters>
-            <controller_manager_name>rb1_robot/controller_manager</controller_manager_name>
-            <ros>
-                <namespace>rb1_robot</namespace>
-                <remapping>/robot_description:=/rb1_robot/robot_description</remapping>
-            </ros>
         </plugin>
     </gazebo>

Commit message: Added a controller for the robot elevator unit

File: cp15_auxiliary_files/rb1_ros2_description/xacro/rb1_ros2_base.urdf.xacro (robot description, xacro)
@@ -97,5 +97,5 @@
         </joint>
     </transmission>
-    <!-- <xacro:ros2_control/> -->
+    <!-- < differential drive controller  /> -->
     <ros2_control name="diff_drive" type="system">
         <hardware>
@@ -121,4 +121,19 @@
         </joint>
     </ros2_control>
+    <!-- < Lifying unit effort controller  /> -->
+    <ros2_control name="lifting_unit_effort_controllers" type="system">
+        <hardware>
+            <plugin>gazebo_ros2_control/GazeboSystem</plugin>
+        </hardware>
+        <joint name="$(arg prefix)elevator_platform_joint">
+            <command_interface name="effort">
+                <param name="min">0</param>
+                <param name="max">10</param>
+            </command_interface>
+            <state_interface name="position"/>
+            <state_interface name="velocity"/>
+            <state_interface name="effort"/>
+        </joint>
+    </ros2_control>
     <!-- Gazebo ros2 control plugins -->
     <gazebo>
@@ -127,3 +142,8 @@
         </plugin>
     </gazebo>
+  <!-- <gazebo>
+    <plugin filename="libgazebo_ros2_control.so" name="gazebo_ros2_control">
+        <parameters>$(find rb1_ros2_description)/config/lifting_unit_effort_controller.yaml</parameters>
+    </plugin>
+  </gazebo> -->
 </robot>
